File: Bluetooth fm transmitter.sch (EAGLE design)
At the start: 19 parts, among them J2 CONNECTOR-8-M5STICKC, U1 BM20SPKA1NBC-0001AA, U2 NS73M_FM_TRANSMITTER, X1 38_KHz

Commit message: Add files via upload
Parts:
- removed J2: CONNECTOR-8-M5STICKC, eagle-library-engr-245-s22:CONNECTOR-8-M5STICKC
- added C1, C2: 15p, eagle-library-engr-245-s22:CAPACITOR-0603
- added C3: 100u, eagle-library-engr-245-s22:CAPACITOR_POLARIZED
- added J1: M5STICKC-PLUS, eagle-library-engr-245-s22:M5STICKC-PLUS
- added MT1, MT2, MT3, MT4: MOUNTING_HOLE-125_250_ROUND, eagle-library-engr-245-s22:MOUNTING_HOLE-125_250_ROUND
- LED3: value Green -> Yellow
- LED4: value (none) -> White
- LED5: value (none) -> Green
- R1, R2: value (none) -> 330R
Connections:
- removed net 5V: R1.2
- new net N$11: C2.1, S2.1, U1.P2_7
- new net N$12: C1.1, S3.1, U1.P0_5
- new net N$13: C1.2, C2.2, S2.2, S3.2
- net 3.3V: now also C3.1, J1.3V3@7, R1.2; no longer J2.3V3@7
- net BAT: now also J1.BAT@6; no longer J2.BAT@6
- net GND: now also C3.2, J1.GND@1; no longer J2.GND@1
- net SDA: now also J1.G36/G25@4; no longer J2.G36/G25@4
- net SDL: now also J1.G26@3; no longer J2.G26@3
- net UNLOCK_DETECT: now also J1.G0@5; no longer J2.G0@5
Other:
- moved on the sheet: S2, S3, X1
